Commit message: j1在极坐标系后半部分，导致角度为-pi，余弦定理论求出的理论长度错误

File: src/solver/arm/zyz_ik/urdf/6axis_arm.urdf (robot description, URDF)
Before this commit: robot 6axis_arm, 8 links, 7 joints
Joints:
- joint joint_4: origin xyz= -0.055 0.3783 0   rpy=-1.5708 0 0 -> xyz= 0 0.0183 0   rpy=-1.5708 0 0
- joint joint_5: origin xyz=0 0 0 rpy=1.5708 0 0 -> xyz=0 0 0.32 rpy=1.5708 0 0
- joint joint_6: origin xyz= 0 0 0 rpy=-1.5708 0 0 -> xyz= 0 0.05 0 rpy=-1.5708 0 0
